Commit message: robot falling in gazebo fix

File: humanoid_description/urdf/humanoid.gazebo.xacro (robot description, xacro)
@@ -2,5 +2,6 @@
 <robot xmlns:xacro="http://www.ros.org/wiki/xacro">
     <gazebo>
-        <plugin filename="ign_gazebo_joint_state_publisher_system" name="gz::sim::systems::JointStatePublisher">            <topic>joint_states</topic>
+        <plugin filename="ign_gazebo_joint_state_publisher_system" name="gz::sim::systems::JointStatePublisher">
+            <topic>joint_states</topic>
             <update_rate>50</update_rate>
         </plugin>

File: humanoid_description/urdf/humanoid.xacro (robot description, xacro)
@@ -421,6 +421,6 @@
         <child link="pelvic-to-chest_link"/>
         <!-- prismatic adds: Prevents math crashes by setting motion bounds (in meters)  -->
-        <axis xyz="0 1 0"/>
-        <limit lower="-1.0" upper="1.0" effort="10.0" velocity="1.0"/>
+        <!-- <axis xyz="0 1 0"/>
+        <limit lower="-1.0" upper="1.0" effort="10.0" velocity="1.0"/> -->
     </joint>
     <link name="pelvic-to-chest_link">
@@ -460,11 +460,11 @@
             <origin xyz="-0.343943 0.125478 -0.38665" rpy="1.570796 0.0 0.0"/>
             <geometry>
-                <mesh filename="package://humanoid_description/meshes/torso_to_femur.STL" scale="0.001 0.001 0.001"/>
-            </geometry>
-        </visual>
-        <collision>
-            <origin xyz="-0.343943 0.125478 -0.38665" rpy="1.570796 0.0 0.0"/>
-            <geometry>
-                <mesh filename="package://humanoid_description/meshes/torso_to_femur.STL" scale="0.001 0.001 0.001"/>
+                <mesh filename="package://humanoid_description/meshes/left-torso_to_femur.STL" scale="0.001 0.001 0.001"/>
+            </geometry>
+        </visual>
+        <collision>
+            <origin xyz="-0.343943 0.125478 -0.38665" rpy="1.570796 0.0 0.0"/>
+            <geometry>
+                <mesh filename="package://humanoid_description/meshes/left-torso_to_femur.STL" scale="0.001 0.001 0.001"/>
             </geometry>
         </collision>
@@ -475,5 +475,5 @@
         <child link="pelvic-to-rightleg_link"/>
         <!-- prismatic adds: Prevents math crashes by setting motion bounds (in meters)  -->
-        <!-- <axis xyz="1 0 0"/>
+        <!-- <axis xyz="0 1 0"/>
         <limit lower="-1.0" upper="1.0" effort="10.0" velocity="1.0"/> -->
     </joint>
@@ -485,16 +485,35 @@
         </inertial>
         <visual>
-            <origin xyz="0.343943 -0.125478 -0.38665" rpy="1.570796 0.0 3.14159"/>
-            <geometry>
-                <mesh filename="package://humanoid_description/meshes/torso_to_femur.STL" scale="0.001 0.001 0.001"/>
-            </geometry>
-        </visual>
-        <collision>
-            <origin xyz="0.343943 -0.125478 -0.38665" rpy="1.570796 0.0 3.14159"/>
-            <geometry>
-                <mesh filename="package://humanoid_description/meshes/torso_to_femur.STL" scale="0.001 0.001 0.001"/>
-            </geometry>
-        </collision>
-    </link>
+            <origin xyz="0.197943 -0.011478 -0.38665" rpy="1.570796 0.0 3.14159"/>
+            <geometry>
+                <mesh filename="package://humanoid_description/meshes/left-torso_to_femur.STL" scale="0.001 0.001 0.001"/>
+            </geometry>
+        </visual>
+        <collision>
+            <origin xyz="0.197943 -0.011478 -0.38665" rpy="1.570796 0.0 3.14159"/>
+            <geometry>
+                <mesh filename="package://humanoid_description/meshes/left-torso_to_femur.STL" scale="0.001 0.001 0.001"/>
+            </geometry>
+        </collision>
+    </link>
+    <!-- <link name="pelvic-to-rightleg_link"> exchanged-not straight
+        <inertial>
+            <origin xyz="0.0 0.0 0.0" rpy="0.0 0.0 0.0"/>
+            <mass value="15.0"/>
+            <inertia ixx="0.1" ixy="0.0" ixz="0.0" iyy="0.1" iyz="0.0" izz="0.1"/>
+        </inertial>
+        <visual>
+            <origin xyz="-0.343943 0.125478 -0.38665" rpy="1.570796 0.0 0.0"/>
+            <geometry>
+                <mesh filename="package://humanoid_description/meshes/right-torso_to_femur.STL" scale="0.001 0.001 0.001"/>
+            </geometry>
+        </visual>
+        <collision>
+            <origin xyz="-0.343943 0.125478 -0.38665" rpy="1.570796 0.0 0.0"/>
+            <geometry>
+                <mesh filename="package://humanoid_description/meshes/right-torso_to_femur.STL" scale="0.001 0.001 0.001"/>
+            </geometry>
+        </collision>
+    </link> -->
     <joint name="torso-to-leftleg_joint" type="fixed">
         <origin xyz="0.0 0.0 0.0" rpy="0.0 0.0 0.0"/>
@@ -512,5 +531,5 @@
         </inertial>
         <visual>
-            <origin xyz="-0.343943 0.125478 -0.38665" rpy="1.570796 0.0 0.0"/>
+            <origin xyz="0.500943 -0.066478 -0.40265" rpy="1.570796 0.0 3.14159"/>
             <geometry>
                 <mesh filename="package://humanoid_description/meshes/Waist_to_knee.STL" scale="0.001 0.001 0.001"/>
@@ -518,5 +537,5 @@
         </visual>
         <collision>
-            <origin xyz="-0.343943 0.125478 -0.38665" rpy="1.570796 0.0 0.0"/>
+            <origin xyz="0.500943 -0.066478 -0.40265" rpy="1.570796 0.0 3.14159"/>
             <geometry>
                 <mesh filename="package://humanoid_description/meshes/Waist_to_knee.STL" scale="0.001 0.001 0.001"/>
@@ -539,5 +558,5 @@
         </inertial>
         <visual>
-            <origin xyz="0.343943 -0.125478 -0.38665" rpy="1.570796 0.0 3.14159"/>
+            <origin xyz="0.268943 -0.066478 -0.40265" rpy="1.570796 0.0 3.14159"/>
             <geometry>
                 <mesh filename="package://humanoid_description/meshes/Waist_to_knee.STL" scale="0.001 0.001 0.001"/>
@@ -545,5 +564,5 @@
         </visual>
         <collision>
-            <origin xyz="0.343943 -0.125478 -0.38665" rpy="1.570796 0.0 3.14159"/>
+            <origin xyz="0.268943 -0.066478 -0.40265" rpy="1.570796 0.0 3.14159"/>
             <geometry>
                 <mesh filename="package://humanoid_description/meshes/Waist_to_knee.STL" scale="0.001 0.001 0.001"/>
@@ -556,5 +575,5 @@
         <child link="leftknee-to-ankle_link"/>
         <!-- prismatic adds: Prevents math crashes by setting motion bounds (in meters)  -->
-        <!-- <axis xyz="1 0 0"/>
+        <!-- <axis xyz="0 1 0"/>
         <limit lower="-1.0" upper="1.0" effort="10.0" velocity="1.0"/> -->
     </joint>
@@ -566,13 +585,13 @@
         </inertial>
         <visual>
-            <origin xyz="-0.343943 0.125478 -0.38665" rpy="1.570796 0.0 0.0"/>
-            <geometry>
-                <mesh filename="package://humanoid_description/meshes/Knee_to_Ankle.STL" scale="0.001 0.001 0.001"/>
-            </geometry>
-        </visual>
-        <collision>
-            <origin xyz="-0.343943 0.125478 -0.38665" rpy="1.570796 0.0 0.0"/>
-            <geometry>
-                <mesh filename="package://humanoid_description/meshes/Knee_to_Ankle.STL" scale="0.001 0.001 0.001"/>
+            <origin xyz="0.195943 0.022478 -0.38665" rpy="1.440796 0.0 3.14159"/>
+            <geometry>
+                <mesh filename="package://humanoid_description/meshes/leftKnee_to_Ankle.STL" scale="0.001 0.001 0.001"/>
+            </geometry>
+        </visual>
+        <collision>
+            <origin xyz="0.195943 0.022478 -0.38665" rpy="1.440796 0.0 3.14159"/>
+            <geometry>
+                <mesh filename="package://humanoid_description/meshes/leftKnee_to_Ankle.STL" scale="0.001 0.001 0.001"/>
             </geometry>
         </collision>
@@ -593,13 +612,13 @@
         </inertial>
         <visual>
-            <origin xyz="0.343943 -0.125478 -0.38665" rpy="1.570796 0.0 3.14159"/>
-            <geometry>
-                <mesh filename="package://humanoid_description/meshes/Knee_to_Ankle.STL" scale="0.001 0.001 0.001"/>
-            </geometry>
-        </visual>
-        <collision>
-            <origin xyz="0.343943 -0.125478 -0.38665" rpy="1.570796 0.0 3.14159"/>
-            <geometry>
-                <mesh filename="package://humanoid_description/meshes/Knee_to_Ankle.STL" scale="0.001 0.001 0.001"/>
+            <origin xyz="0.195943 0.015522 -0.38665" rpy="1.440796 0.0 3.14159"/>
+            <geometry>
+                <mesh filename="package://humanoid_description/meshes/rightKnee_to_Ankle.STL" scale="0.001 0.001 0.001"/>
+            </geometry>
+        </visual>
+        <collision>
+            <origin xyz="0.195943 0.015522 -0.38665" rpy="1.440796 0.0 3.14159"/>
+            <geometry>
+                <mesh filename="package://humanoid_description/meshes/rightKnee_to_Ankle.STL" scale="0.001 0.001 0.001"/>
             </geometry>
         </collision>
@@ -610,5 +629,5 @@
         <child link="leftankle-to-feet_link"/>
         <!-- prismatic adds: Prevents math crashes by setting motion bounds (in meters)  -->
-        <!-- <axis xyz="1 0 0"/>
+        <!-- <axis xyz="0 1 0"/>
         <limit lower="-1.0" upper="1.0" effort="10.0" velocity="1.0"/> -->
     </joint>
@@ -620,13 +639,13 @@
         </inertial>
         <visual>
-            <origin xyz="-0.343943 0.125478 -0.38665" rpy="1.570796 0.0 0.0"/>
-            <geometry>
-                <mesh filename="package://humanoid_description/meshes/Foot.STL" scale="0.001 0.001 0.001"/>
-            </geometry>
-        </visual>
-        <collision>
-            <origin xyz="-0.343943 0.125478 -0.38665" rpy="1.570796 0.0 0.0"/>
-            <geometry>
-                <mesh filename="package://humanoid_description/meshes/Foot.STL" scale="0.001 0.001 0.001"/>
+            <origin xyz="-0.343943 0.081978 -0.38285" rpy="1.532796 0.0 0.0"/>
+            <geometry>
+                <mesh filename="package://humanoid_description/meshes/left_foot.STL" scale="0.001 0.001 0.001"/>
+            </geometry>
+        </visual>
+        <collision>
+            <origin xyz="-0.343943 0.081978 -0.38285" rpy="1.532796 0.0 0.0"/>
+            <geometry>
+                <mesh filename="package://humanoid_description/meshes/left_foot.STL" scale="0.001 0.001 0.001"/>
             </geometry>
         </collision>
@@ -637,5 +656,5 @@
         <child link="rightankle-to-feet_link"/>
         <!-- prismatic adds: Prevents math crashes by setting motion bounds (in meters)  -->
-        <!-- <axis xyz="1 0 0"/>
+        <!-- <axis xyz="0 1 0"/>
         <limit lower="-1.0" upper="1.0" effort="10.0" velocity="1.0"/> -->
     </joint>
@@ -647,13 +666,13 @@
         </inertial>
         <visual>
-            <origin xyz="-0.57343 0.071478 -0.38665" rpy="1.570796 0.0 0.0"/>
-            <geometry>
-                <mesh filename="package://humanoid_description/meshes/Foot.STL" scale="0.001 0.001 0.001"/>
-            </geometry>
-        </visual>
-        <collision>
-            <origin xyz="-0.343943 -0.125478 -0.38665" rpy="1.570796 0.0 0.0"/>
-            <geometry>
-                <mesh filename="package://humanoid_description/meshes/Foot.STL" scale="0.001 0.001 0.001"/>
+            <origin xyz="-0.343943 0.081978 -0.38285" rpy="1.532796 0.0 0.0"/>
+            <geometry>
+                <mesh filename="package://humanoid_description/meshes/right_foot.STL" scale="0.001 0.001 0.001"/>
+            </geometry>
+        </visual>
+        <collision>
+            <origin xyz="-0.343943 0.081978 -0.38285" rpy="1.532796 0.0 0.0"/>
+            <geometry>
+                <mesh filename="package://humanoid_description/meshes/right_foot.STL" scale="0.001 0.001 0.001"/>
             </geometry>
         </collision>
